File: K3PRO.kicad_sch (KiCad schematic)
At the start: 34 parts, among them J1 USB_C_Receptacle_USB2.0, J2 TESTPOINT STM32, K1 SW_SPDT, P01 TestPoint, Q1 NMOS, Q2 NMOS, Q4 NMOS, U6 STM32L432KBUx

Commit message: Output PDF
Other:
- title: (none) -> Keychron K3 Pro
Changed lines of the file:
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@@
 (kicad_sch (version 20230121) (generator eeschema)
   (paper "A4")
+  (title_block
+    (title "Keychron K3 Pro")
+    (date "2023-07-04")
+  )
   (junction (at 190.5 81.28) (diameter 0) (color 0 0 0 0)
   )
