File: K3PRO_BT.kicad_sch (KiCad schematic)
At the start: 12 parts, among them J3 Conn_01x04, U4 MODULE_CYW20730, U9 EEPROM (NC)

Commit message: Output PDF
Other:
- title: (none) -> Keychron K3 Pro
Changed lines of the file:
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@@
 (kicad_sch (version 20230121) (generator eeschema)
   (paper "A4")
+  (title_block
+    (title "Keychron K3 Pro")
+    (date "2023-07-04")
+  )
   (junction (at 215.9 50.8) (diameter 0) (color 0 0 0 0)
   )
