File: K3PRO_LEDS.kicad_sch (KiCad schematic)
At the start: 23 parts, among them U4 CKLED2001, U5 CKLED2001

Commit message: Output PDF
Parts:
- removed RGB1, RGB2, RGB3, RGB4: LED_ARGB, symbol Device:LED_ARGB
Other:
- note added: "太累了，自己测吧"
- title: (none) -> Keychron K3 Pro
Changed lines of the file:
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@@
 (kicad_sch (version 20230121) (generator eeschema)
   (paper "A4")
+  (title_block
+    (title "Keychron K3 Pro")
+    (date "2023-07-04")
+  )
   (junction (at 187.96 152.4) (diameter 0) (color 0 0 0 0)
   )
@@
   (junction (at 111.76 177.8) (diameter 0) (color 0 0 0 0)
   )
-  (junction (at 22.86 15.24) (diameter 0) (color 0 0 0 0)
-  )
-  (junction (at 20.32 15.24) (diameter 0) (color 0 0 0 0)
-  )
   (junction (at 187.96 139.7) (diameter 0) (color 0 0 0 0)
   )
@@
   )
   (junction (at 226.06 139.7) (diameter 0) (color 0 0 0 0)
-  )
-  (junction (at 17.78 15.24) (diameter 0) (color 0 0 0 0)
   )
   (no_connect (at 78.74 185.42))
@@
     (stroke (width 0) (type default))
   )
-  (wire (pts (xy 20.32 30.48) (xy 22.86 30.48))
-    (stroke (width 0) (type default))
-  )
   (wire (pts (xy 106.68 175.26) (xy 106.68 180.34))
     (stroke (width 0) (type default))
@@
     (stroke (width 0) (type default))
   )
-  (wire (pts (xy 20.32 15.24) (xy 20.32 30.48))
-    (stroke (width 0) (type default))
-  )
-  (wire (pts (xy 15.24 17.78) (xy 139.7 17.78))
-    (stroke (width 0) (type default))
-  )
   (wire (pts (xy 187.96 139.7) (xy 187.96 142.24))
     (stroke (width 0) (type default))
@@
     (stroke (width 0) (type default))
   )
-  (wire (pts (xy 20.32 15.24) (xy 22.86 15.24))
-    (stroke (width 0) (type default))
-  )
-  (wire (pts (xy 15.24 40.64) (xy 88.9 40.64))
-    (stroke (width 0) (type default))
-  )
   (wire (pts (xy 30.48 175.26) (xy 30.48 179.07))
     (stroke (width 0) (type default))
@@
     (stroke (width 0) (type default))
   )
-  (wire (pts (xy 17.78 15.24) (xy 20.32 15.24))
-    (stroke (width 0) (type default))
-  )
-  (wire (pts (xy 15.24 15.24) (xy 17.78 15.24))
-    (stroke (width 0) (type default))
-  )
-  (wire (pts (xy 22.86 15.24) (xy 22.86 25.4))
-    (stroke (width 0) (type default))
-  )
-  (wire (pts (xy 17.78 35.56) (xy 22.86 35.56))
-    (stroke (width 0) (type default))
-  )
-  (wire (pts (xy 22.86 15.24) (xy 139.7 15.24))
-    (stroke (width 0) (type default))
-  )
   (wire (pts (xy 177.8 152.4) (xy 187.96 152.4))
     (stroke (width 0) (type default))
   )
-  (wire (pts (xy 15.24 43.18) (xy 88.9 43.18))
-    (stroke (width 0) (type default))
-  )
   (wire (pts (xy 45.72 177.8) (xy 48.26 177.8))
     (stroke (width 0) (type default))
   )
-  (wire (pts (xy 17.78 15.24) (xy 17.78 35.56))
-    (stroke (width 0) (type default))
-  )
   (wire (pts (xy 20.32 175.26) (xy 30.48 175.26))
     (stroke (width 0) (type default))
   )
-  (wire (pts (xy 15.24 45.72) (xy 88.9 45.72))
-    (stroke (width 0) (type default))
-  )
-  (wire (pts (xy 15.24 20.32) (xy 139.7 20.32))
-    (stroke (width 0) (type default))
+  (text "太累了，自己测吧" (at 139.7 71.12 0)
+    (effects (font (size 1.27 1.27)) (justify left bottom))
   )
   (label "RGB_EN" (at 177.8 152.4 0) (fields_autoplaced)
@@
         (path "/1c1ad2b2-2251-4ddf-8b29-7fc62f785149/e822a2ca-2b53-4231-b749-172c46d01120"
           (reference "C15") (unit 1)
-        )
-      )
-    )
-  )
-  (symbol (lib_id "Device:LED_ARGB") (at 27.94 30.48 0) (unit 1)
-    (in_bom yes) (on_board yes) (dnp no) (fields_autoplaced)
-    (property "Reference" "RGB1" (at 27.94 19.05 0)
-      (effects (font (size 1.27 1.27)))
-    )
-    (property "Value" "LED_ARGB" (at 27.94 20.32 0)
-      (effects (font (size 1.27 1.27)) hide)
-    )
-    (property "Footprint" "" (at 27.94 31.75 0)
-      (effects (font (size 1.27 1.27)) hide)
-    )
-    (property "Datasheet" "~" (at 27.94 31.75 0)
-      (effects (font (size 1.27 1.27)) hide)
-    )
-    (pin "1")
-    (pin "2")
-    (pin "3")
-    (pin "4")
-    (instances
-      (project "K3PRO"
-        (path "/1c1ad2b2-2251-4ddf-8b29-7fc62f785149/e822a2ca-2b53-4231-b749-172c46d01120"
-          (reference "RGB1") (unit 1)
         )
       )
@@
     )
   )
-  (symbol (lib_id "Device:LED_ARGB") (at 66.04 30.48 0) (unit 1)
-    (in_bom yes) (on_board yes) (dnp no) (fields_autoplaced)
-    (property "Reference" "RGB4" (at 66.04 19.05 0)
-      (effects (font (size 1.27 1.27)))
-    )
-    (property "Value" "LED_ARGB" (at 66.04 20.32 0)
-      (effects (font (size 1.27 1.27)) hide)
-    )
-    (property "Footprint" "" (at 66.04 31.75 0)
-      (effects (font (size 1.27 1.27)) hide)
-    )
-    (property "Datasheet" "~" (at 66.04 31.75 0)
-      (effects (font (size 1.27 1.27)) hide)
-    )
-    (pin "1")
-    (pin "2")
-    (pin "3")
-    (pin "4")
-    (instances
-      (project "K3PRO"
-        (path "/1c1ad2b2-2251-4ddf-8b29-7fc62f785149/e822a2ca-2b53-4231-b749-172c46d01120"
-          (reference "RGB4") (unit 1)
-        )
-      )
-    )
-  )
-  (symbol (lib_id "Device:LED_ARGB") (at 40.64 30.48 0) (unit 1)
-    (in_bom yes) (on_board yes) (dnp no) (fields_autoplaced)
-    (property "Reference" "RGB2" (at 40.64 19.05 0)
-      (effects (font (size 1.27 1.27)))
-    )
-    (property "Value" "LED_ARGB" (at 40.64 20.32 0)
-      (effects (font (size 1.27 1.27)) hide)
-    )
-    (property "Footprint" "" (at 40.64 31.75 0)
-      (effects (font (size 1.27 1.27)) hide)
-    )
-    (property "Datasheet" "~" (at 40.64 31.75 0)
-      (effects (font (size 1.27 1.27)) hide)
-    )
-    (pin "1")
-    (pin "2")
-    (pin "3")
-    (pin "4")
-    (instances
-      (project "K3PRO"
-        (path "/1c1ad2b2-2251-4ddf-8b29-7fc62f785149/e822a2ca-2b53-4231-b749-172c46d01120"
-          (reference "RGB2") (unit 1)
-        )
-      )
-    )
-  )
   (symbol (lib_id "Device:R_US") (at 226.06 146.05 180) (unit 1)
     (in_bom yes) (on_board yes) (dnp no) (fields_autoplaced)
@@
         )
       )
-    )
-  )
-  (symbol (lib_id "Device:LED_ARGB") (at 53.34 30.48 0) (unit 1)
-    (in_bom yes) (on_board yes) (dnp no) (fields_autoplaced)
-    (property "Reference" "RGB3" (at 53.34 19.05 0)
-      (effects (font (size 1.27 1.27)))
-    )
-    (property "Value" "LED_ARGB" (at 53.34 20.32 0)
-      (effects (font (size 1.27 1.27)) hide)
-    )
-    (property "Footprint" "" (at 53.34 31.75 0)
-      (effects (font (size 1.27 1.27)) hide)
-    )
-    (property "Datasheet" "~" (at 53.34 31.75 0)
-      (effects (font (size 1.27 1.27)) hide)
-    )
-    (pin "1")
-    (pin "2")
-    (pin "3")
-    (pin "4")
-    (instances
-      (project "K3PRO"
-        (path "/1c1ad2b2-2251-4ddf-8b29-7fc62f785149/e822a2ca-2b53-4231-b749-172c46d01120"
-          (reference "RGB3") (unit 1)
-        )
-      )
