File: K3PRO_POWER.kicad_sch (KiCad schematic)
At the start: 50 parts, among them K2 SW_SP3T, Q19 NPN, Q20 NPN, Q3 NMOS, U4 TP4056, U5 662K

Commit message: Output PDF
Other:
- title: (none) -> Keychron K3 Pro
Changed lines of the file:
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@@
 (kicad_sch (version 20230121) (generator eeschema)
   (paper "A4")
+  (title_block
+    (title "Keychron K3 Pro")
+    (date "2023-07-04")
+  )
   (junction (at 76.2 30.48) (diameter 0) (color 0 0 0 0)
   )
